File: boards/coupon/coupon.kicad_pcb (KiCad board)
At the start: 2 copper layers, 0 parts

Commit message: Board A layout: deterministic pcbnew build, DRC-clean, golden gerbers
boards/coupon/tools-layout.py rebuilds coupon.kicad_pcb from the
kicad-cli netlist: places all 38 schematic parts + board-only extras,
routes B.Cu single-sided, pours GND, draws the coupon gauges, writes
coupon.kicad_dru, and re-exports byte-stable geometry (KiCad re-mints
UUIDs per run; geometry is deterministic).

Gate state (kicad-cli pcb drc --schematic-parity, KiCad 10.0.4):
0 errors, 0 unconnected, 0 error-level parity. Surviving warnings,
each deliberate: 7 courtyard-class (same-net pad butt-joints R4/S2,
JP5/C1.2, JP5 beside U2's lead-span courtyard; SOIC courtyard overlaps
with C6/C8/R8 at verified >=0.4 pad clearances) -- courtyard checks
downgraded to warning in coupon.kicad_pro with this justification;
18 silk-over-masked-copper cosmetics (zero silk within 0.3 of any
scrubbed aperture); 48 lib bookkeeping (custom coupon:* footprints +
deliberate pad surgery); 1 parity warning (SW1 pad 3 vs flattened
SW_SPDT sub-unit -- netlist proves pin 3 exists, intentionally NC).

Discretionary decisions:
- THT annular >=0.6 law enforced by pad surgery: DIP socket pads
  1.6->2.4x2.0 oval, LED_THT 1.8->2.1, SW_PUSH 2.0->2.3, PAD1/2 drill
  2.0->1.5 (SPEC). Stock CK slide switch (2.0 pitch, 0.35 annular)
  replaced by custom coupon:SW_Slide_SS12D00_HandMill (2.54 pitch,
  2.1/0.9 pads); schematic footprint field updated to match.
- M3 = custom 3.4 NPTH footprint (no stock 3.4) with octagonal
  no-pour/no-track rule areas r3.3.
- Six wire jumpers (Bill 2026-07-29 correction: expected on a
  single-sided milled board): JP1 N_DISCH->S2, JP2+JP3 VCC stitches,
  JP4-JP6 GND into the three pour pockets that flat routing fences
  off. Standard spans 10.16/12.7/15.24, pads 2.1/0.9, board-only,
  net-tie pad groups + the wire modeled as a netted F.Cu track
  (documented exemption: F.Cu is never exported or milled). JP6
  flagged insulated-or-bent in SPEC bench notes.
- GND pour: 0.5 min width, 0.4 clearance, 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
Parts:
- added C1: 10uF, Capacitor_SMD:C_0805_2012Metric_Pad1.18x1.45mm_HandSolder, B.Cu at (119.5, 132.3)
- added C2: 1uF, Capacitor_SMD:C_0603_1608Metric_Pad1.08x0.95mm_HandSolder, B.Cu at (118.0, 124.3)
- added C3: 100nF, Capacitor_SMD:C_0805_2012Metric_Pad1.18x1.45mm_HandSolder, B.Cu at (115.0, 124.2)
- added C4: 10uF, Capacitor_SMD:C_0805_2012Metric_Pad1.18x1.45mm_HandSolder, B.Cu at (140.3, 123.6)
- added C5: 10nF, Capacitor_SMD:C_1206_3216Metric_Pad1.33x1.80mm_HandSolder, B.Cu at (134.3, 128.2)
- added C6: 100nF, Capacitor_SMD:C_0805_2012Metric_Pad1.18x1.45mm_HandSolder, B.Cu at (124.9, 136.9)
- added C7: 100nF, Capacitor_SMD:C_0805_2012Metric_Pad1.18x1.45mm_HandSolder, B.Cu at (132.7, 114.4)
- added C8: 100nF, Capacitor_SMD:C_0805_2012Metric_Pad1.18x1.45mm_HandSolder, B.Cu at (125.9, 130.4)
- added CP1: coupon, R_1206_3216Metric_Pad1.30x1.75mm_HandSolder, B.Cu at (144.7, 138.5)
- added CP2: coupon, R_0805_2012Metric_Pad1.20x1.40mm_HandSolder, B.Cu at (149.0, 138.5)
- added CP3: coupon, R_0603_1608Metric_Pad0.98x0.95mm_HandSolder, B.Cu at (152.7, 138.5)
- added D1: SS14, Diode_SMD:D_SMA_Handsoldering, B.Cu at (115.5, 128.0)
- added H1: , coupon:MountingHole_3.4mm_NPTH, F.Cu at (104.5, 104.5)
- added H2: , coupon:MountingHole_3.4mm_NPTH, F.Cu at (150.5, 104.5)
- added H3: , coupon:MountingHole_3.4mm_NPTH, F.Cu at (104.5, 135.5)
- added H4: , coupon:MountingHole_3.4mm_NPTH, F.Cu at (150.5, 135.5)
- added JP1: wire 10.16mm, coupon:JumperWire_P10.16mm, F.Cu at (142.5, 111.2)
- added JP2: wire 12.7mm, coupon:JumperWire_P12.7mm, F.Cu at (119.3, 119.0)
- added JP3: wire 15.24mm, coupon:JumperWire_P15.24mm, F.Cu at (124.1, 109.9)
- added JP4: wire 15.24mm, coupon:JumperWire_P15.24mm, F.Cu at (129.6, 112.7)
- added JP5: wire 12.7mm, coupon:JumperWire_P12.7mm, F.Cu at (131.5, 136.0)
- added JP6: wire 10.16mm, coupon:JumperWire_P10.16mm, F.Cu at (123.3, 128.3)
- added L1: 10uH, Inductor_SMD:L_0805_2012Metric_Pad1.05x1.20mm_HandSolder, B.Cu at (121.0, 126.2)
- added LED1: LED_RED, LED_SMD:LED_0805_2012Metric_Pad1.15x1.40mm_HandSolder, B.Cu at (110.5, 120.8)
- added LED2: LED_5MM, LED_THT:LED_D5.0mm, F.Cu at (124.0, 105.5)
- added LED3: LED_5MM, LED_THT:LED_D5.0mm, F.Cu at (132.0, 105.5)
- added LED4: LED_GRN, LED_SMD:LED_0805_2012Metric_Pad1.15x1.40mm_HandSolder, B.Cu at (139.6, 137.9)
- added PAD1: +5V, TestPoint:TestPoint_THTPad_D4.0mm_Drill2.0mm, F.Cu at (104.8, 122.5)
- added PAD2: GND, TestPoint:TestPoint_THTPad_D4.0mm_Drill2.0mm, F.Cu at (104.8, 129.5)
- added Q1: S8050, Package_TO_SOT_SMD:SOT-23_Handsoldering, B.Cu at (117.5, 110.0)
- added R1: 1k, Resistor_SMD:R_1206_3216Metric_Pad1.30x1.75mm_HandSolder, B.Cu at (110.5, 116.3)
- added R10: 10k, Resistor_SMD:R_0805_2012Metric_Pad1.20x1.40mm_HandSolder, B.Cu at (122.0, 134.6)
- added R11: 330R, Resistor_SMD:R_1206_3216Metric_Pad1.30x1.75mm_HandSolder, B.Cu at (137.3, 136.4)
- added R2: 10k, Resistor_SMD:R_0603_1608Metric_Pad0.98x0.95mm_HandSolder, B.Cu at (137.0, 114.5)
- added R3: 33k, Resistor_SMD:R_0805_2012Metric_Pad1.20x1.40mm_HandSolder, B.Cu at (138.0, 120.0)
- added R4: 6.8k, Resistor_SMD:R_1206_3216Metric_Pad1.30x1.75mm_HandSolder, B.Cu at (138.0, 123.6)
- added R5: 1k, Resistor_SMD:R_0603_1608Metric_Pad0.98x0.95mm_HandSolder, B.Cu at (121.5, 111.9)
- added R6: 330R, Resistor_SMD:R_0805_2012Metric_Pad1.20x1.40mm_HandSolder, B.Cu at (127.8, 109.6)
- added R7: 330R, Resistor_SMD:R_1206_3216Metric_Pad1.30x1.75mm_HandSolder, B.Cu at (135.8, 109.6)
- added R8: 100k, Resistor_SMD:R_0603_1608Metric_Pad0.98x0.95mm_HandSolder, B.Cu at (128.7, 129.6)
- added R9: 10k, Resistor_SMD:R_0603_1608Metric_Pad0.98x0.95mm_HandSolder, B.Cu at (123.7, 133.7)
- added S2: SW_Push, Button_Switch_THT:SW_PUSH_6mm, F.Cu at (142.5, 125.7)
- added SW1: SW_SPDT, coupon:SW_Slide_SS12D00_HandMill, F.Cu at (109.5, 128.0)
- added TP1: TestPoint, TestPoint:TestPoint_Pad_D2.0mm, B.Cu at (144.9, 109.8)
- added TP2: TestPoint, TestPoint:TestPoint_Pad_D2.0mm, B.Cu at (153.1, 109.8)
- added TP3: TestPoint, TestPoint:TestPoint_Pad_D2.0mm, B.Cu at (144.9, 115.4)
- added TP4: TestPoint, TestPoint:TestPoint_Pad_D2.0mm, B.Cu at (153.1, 115.4)
- added TP5: TestPoint, TestPoint:TestPoint_Pad_D2.0mm, B.Cu at (144.9, 120.5)
- added TP6: TestPoint, TestPoint:TestPoint_Pad_D2.0mm, B.Cu at (153.1, 120.5)
- added U1: NE555P, Package_DIP:DIP-8_W7.62mm_Socket, F.Cu at (126.0, 117.5)
- added U2: LM358, Package_SO:SOIC-8_3.9x4.9mm_P1.27mm, B.Cu at (128.2, 133.5)
Routing:
- net VCC: track 0.00 -> 87.9 mm
- net /LADDER_040: track 0.00 -> 39.7 mm
- net GND: track 0.00 -> 38.4 mm
- net /N_DISCH: track 0.00 -> 38.2 mm
- net /LADDER_050: track 0.00 -> 33.4 mm
- net /LADDER_060: track 0.00 -> 25.6 mm
- net /TRIG_THR: track 0.00 -> 25.0 mm
- net /LEDK: track 0.00 -> 22.7 mm
- net /VHALF: track 0.00 -> 22.6 mm
- net /BLINK: track 0.00 -> 12.9 mm
- net /N_U2AOUT: track 0.00 -> 9.48 mm
- net /VF: track 0.00 -> 6.93 mm
- net /N_KICK: track 0.00 -> 6.55 mm
- net /N_LED2A: track 0.00 -> 6.31 mm
- net /VIN: track 0.00 -> 5.79 mm
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- added copper zone on B.Cu, net GND
Other:
- board outline added: 55 x 40 mm
- rule pad_to_mask_clearance: 0.05 -> 0
- board text added: "+5V"
- board text added: "0.4"
- board text added: "0.5"
- board text added: "0.6"
- board text added: "2026-07"
- board text added: "COUPON v1"
- board text added: "GND"
- board text added: "SILK 1.2"
- board text added: "SILK 1.5"
- board text added: "SILK 2.0"
