File: boards/coupon/coupon.kicad_pcb (KiCad board)
At the start: 2 copper layers, 55 x 40 mm, 51 parts, among them Q1 S8050, SW1 SW_SPDT, U1 NE555P, U2 LM358

Commit message: Board A learns the fab houses' manners: thermals, necks, and three new laws
The operator's render review, second half: solid pour contact heat-sinks
a hand iron, and the big fab houses' DFM was to be incorporated
(guides/pcb-dfm-notes.md). Board-side and gate-side land together
because the gap-band check would rightly have failed the old board.

Board (tools-layout.py, DRC 0 errors with --severity-all
--schematic-parity): thermal reliefs on hole-centered GND pads (gap
0.4, spoke 0.6 x4 @ 45deg; U1.1 at 90 -- the corner socket pin's
diagonals died in the BLINK moat); SMD GND pads ZONE_CONNECTION_NONE
with one routed 0.6 neck each; teardrops at 15 THT junctions; a
build-time >=90deg copper-turn assertion (caught /VF at 95.3deg and
both N_LED diagonals on first run); silk floor 1.0 + a SILK 1.0 ladder
rung; the lead+0.2..0.4 hole rule (the 0.8 plunge-only class is
extinct: 39 bores in {0.9, 1.1, 1.5, 3.4}); U2's 0.60 SOIC pads
widened to 0.80; LED2/3 and C6 moved off the tab stubs; mask expansion
0 asserted.

Killing solid connects re-plumbed GND: pockets stitched through solid
pads lost their path to ground. JP6 grew 10.16->12.7 so its far pad
lands in MAIN pour; JP7 (the seventh jumper) bridges the pocket that
TRIG's limb, N_KICK, S2's moat and N_U2AOUT seal exactly shut. The
jumper 1.0-drill class was tried and REVERTED (2.2 pads shaved three
0.44 clearances under the 0.4 law) -- recorded in make_jumper.

Gate (checks.py): thermal solid connect / spoke count / spoke width
(pour = flooded component >=25% of ink AND >=50mm2 -- the twosided
fixture taught that a bare pad on a tiny board clears a fraction
test); pad scrubbability >=0.70 (the OLD golden board failed it on U2
at first contact); silk text height >=1.0, stroke ratio 1:7.5..1:3.5,
glyph gap >=0.15 TRUE ink distance (the 0.3 aspiration exceeds KiCad's
font -- measured 0.150 at h1.5; JLCPCB's floor is the bar, the SILK
1.0 rung is the bloom gauge). Three caught negatives on corrupted
copies of the blessed rast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
Parts:
- added JP7: wire 12.7mm, coupon:JumperWire_P12.7mm, F.Cu at (141.5, 135.0)
- JP6: value wire 10.16mm -> wire 12.7mm; footprint coupon:JumperWire_P10.16mm -> coupon:JumperWire_P12.7mm
- moved C6 2.07 mm to (122.9, 137.4), turned to 180 degrees
- moved LED2 0.85 mm to (124.0, 106.3)
- moved LED3 0.85 mm to (132.0, 106.3)
- turned JP6 to -170.95 degrees
- turned R10 to 90 degrees
Routing:
- net GND: track 38.4 -> 87.5 mm
- net /N_DISCH: track 38.2 -> 59.3 mm
- net /LEDK: track 22.7 -> 33.0 mm
- net /TRIG_THR: track 25.0 -> 33.8 mm
- net VCC: track 87.9 -> 96.6 mm
- net /N_KICK: track 6.55 -> 15.1 mm
- net /VIN_SW: track 3.50 -> 7.86 mm
- net /VIN: track 5.79 -> 10.1 mm
- net /N_LED2A: track 6.31 -> 3.51 mm
- net /N_LED3A: track 5.76 -> 2.96 mm
Other:
- board text added: "SILK 1.0"
