File: boards/coupon/coupon.kicad_pcb (KiCad board)
At the start: 2 copper layers, 55 x 40 mm, 52 parts, among them Q1 S8050, SW1 SW_SPDT, U1 NE555P, U2 LM358

Commit message: The silk auto-labeler: 41 of 48 parts named, and no hand ever places a label
boards/silklabel.py — pure-geometry, deterministic, called by layout
scripts at build time. The gate's laws are candidate rejection: mask
apertures + 0.40 (the clip law plus slack), silk + 0.20, edge 1.00,
labels + 0.30, and precise keep-clears (the three serpentine blocks the
loupe reads, the M3 washer shadows). Board A taught the tuning, each
step measured: soft courtyards (hard = 12/48), slide-along-edge slots,
far gap tiers, re-seat sweeps + depth-1 eviction to fixpoint. The seven
unplaced are printed, reasoned, and stay off the board: TP2/4/6 could
only label the serpentines, CP3 is cornered, CP2/S2/U2 lose an
over-subscribed neighbourhood.

Closure: DRC 0, raster diff shows Cu/Mask/Paste/drl untouched and silk
strictly additive; gate PASS x4; mill/scrub/holes byte-identical to
golden; silk re-blessed 536 -> 1562 strokes.

Co-Authored-By: Claude Fable 5 <noreply@anthropic.com>
Claude-Session: https://claude.ai/code/session_0195F1eYbZrSx79t6f85WiNq
Other:
- board text added: "C1"
- board text added: "C2"
- board text added: "C3"
- board text added: "C4"
- board text added: "C5"
- board text added: "C6"
- board text added: "C7"
- board text added: "C8"
- board text added: "CP1"
- board text added: "D1"
- board text added: "JP1"
- board text added: "JP2"
- board text added: "JP3"
- board text added: "JP4"
- board text added: "JP5"
- board text added: "JP6"
- board text added: "JP7"
- board text added: "L1"
- board text added: "LED1"
- board text added: "LED2"
- board text added: "LED3"
- board text added: "LED4"
- board text added: "PAD1"
- board text added: "PAD2"
- board text added: "Q1"
- board text added: "R1"
- board text added: "R10"
- board text added: "R11"
- board text added: "R2"
- board text added: "R3"
- board text added: "R4"
- board text added: "R5"
- board text added: "R6"
- board text added: "R7"
- board text added: "R8"
- board text added: "R9"
- board text added: "SW1"
- board text added: "TP1"
- board text added: "TP3"
- board text added: "TP5"
- board text added: "U1"
